Commit message: D-481: IKA URDF kutle/atalet duzeltildi (kaba tahmin) + kok neden kesinlendi
Kullanicinin paylastigi SolidWorks "Montaj6v2v20" mass properties ekran
goruntusu kok nedeni kesinledi: montaj seviyesinde elle girilmis kutle
gecersiz kilma (9308 g, DDR tahminini yansitiyordu) URDF disa
aktariminda HER baga (govde+4 teker) aynen kopyalanmis.

Duzeltme: govde 9.308->6.907 kg, her teker 9.308->0.1632 kg (BOM
oranlariyla dagitilip gercek tartima 7.56 kg olceklendi, D-478/D-480).
Atalet tensoru ayni oranla olceklendi - KABA TAHMIN, CAD'den yeniden
hesaplanmadi, dosya ici yorumla acikca etiketlendi. CoM konumuna
dokunulmadi (T262 - montaj CoM'u Z=1019mm gosteriyor ama zarf 310mm,
ayri bir CAD sorunu). CSV bilerek degistirilmedi (ham kanit kaydi).

Dogrulama: gz sdf -p (gercek Gazebo11) XML gecerli, toplam 7.5598 kg.

File: IKA_GAZEBO_MODEL/urdf/IKA_GAZEBO_MODEL.urdf (robot description, URDF)
Before this commit: robot IKA_GAZEBO_MODEL, 6 links, 5 joints
Links:
- link base_link: mass 9.308 -> 6.907
- link sag_arka_teker: mass 9.308 -> 0.1632
- link sag_on_teker: mass 9.308 -> 0.1632
- link sol_arka_teker: mass 9.308 -> 0.1632
- link sol_on_teker: mass 9.308 -> 0.1632
